File: EAGLE/battleship.brd (EAGLE design)
At the start: 120 x 90 mm, 21 parts, among them IC1 EK-TM4C123GXLP

Commit message: update eagle files
Parts:
- added JP10, JP7, JP8, JP9: (no value), pinhead:1X10
- added JP11, JP12, JP13: (no value), pinhead:2X10
- moved LS1 20.4 mm to (7.62, 29.2)
- moved R4 6.35 mm to (19.1, 80.0)
- moved R1 2.54 mm to (19.1, 6.35)
- moved R2 2.54 mm to (19.1, 10.2)
- moved R3 2.54 mm to (19.1, 14.0)
- moved RIGHT 2.54 mm to (29.2, 61.0)
- moved LEFT 1.27 mm to (10.2, 61.0)
- moved UP 1.27 mm to (19.1, 68.6)
Connections:
- removed net N$3: IC1.1, JP3.1
- new net 3.3V: IC1.1, JP1.6, JP10.1, JP2.6, JP3.1, X1.4
- new net CE: JP1.2, JP2.2
- new net CLK: JP1.5, JP2.5
- new net DC: JP1.3, JP2.3
- new net DIN: JP1.4, JP2.4
- new net LIGHT: JP1.7, JP2.7
- new net N$52: JP11.3, JP11.4, JP12.3, JP12.4, JP13.3, JP13.4
- new net N$53: X1.2
- new net N$54: X1.3
- new net N$55: JP11.7, JP11.8, JP12.7, JP12.8, JP13.7, JP13.8
- new net N$58: JP11.11, JP11.12, JP12.11, JP12.12, JP13.11, JP13.12
- new net N$60: JP11.15, JP11.16, JP12.15, JP12.16, JP13.15, JP13.16
- new net N$61: JP11.17, JP11.18, JP12.17, JP12.18, JP13.17, JP13.18
- new net N$62: JP11.19, JP11.20, JP12.19, JP12.20, JP13.19, JP13.20
- new net N$73: JP11.1, JP11.2, JP12.1, JP12.2, JP13.1, JP13.2
- new net N$76: JP11.5, JP11.6, JP12.5, JP12.6, JP13.5, JP13.6
- new net N$77: JP11.10, JP11.9, JP12.10, JP12.9, JP13.10, JP13.9
- new net N$79: JP11.13, JP11.14, JP12.13, JP12.14, JP13.13, JP13.14
- new net RESET: JP1.1, JP2.1
- net GND: now also JP1.8, JP2.8, JP7.1, JP9.2, X1.1
- net N$10: now also JP10.10
- net N$11: now also JP7.10
- net N$12: now also JP7.9
- net N$13: now also JP7.8
- net N$14: now also JP7.7
- net N$15: now also JP7.6
- net N$16: now also JP7.5
- net N$17: now also JP7.4
- net N$18: now also JP7.3
- net N$19: now also JP7.2
- net N$21: now also JP9.1
- net N$23: now also JP9.3
- net N$24: now also JP9.4
- net N$25: now also JP9.8
- net N$26: now also JP9.9
- net N$27: now also JP9.10
- net N$28: now also JP8.10
- net N$29: now also JP8.9
- net N$30: now also JP8.8
- net N$31: now also JP8.7
- net N$32: now also JP8.6
- net N$33: now also JP8.5
- net N$34: now also JP8.4
- net N$35: now also JP8.3
- net N$36: now also JP8.2
- net N$37: now also JP8.1
- net N$38: now also JP10.6
- net N$39: now also JP9.7
- net N$4: now also JP10.2
- net N$40: now also JP10.7
- net N$41: now also JP9.6
- net N$42: now also JP9.5
- net N$5: now also JP10.3
- net N$6: now also JP10.4
- net N$7: now also JP10.5
- net N$8: now also JP10.8
- net N$9: now also JP10.9

Commit message: update eagle files
Parts:
- removed JP10, JP6, JP7, JP8, JP9: (no value), pinhead:1X10
- added JP14: (no value), pinhead:2X10
- JP3, JP4, JP5: device pinhead:1X10 -> pinhead:2X10
- moved JP4 30.5 mm to (45.7, 15.2)
- moved R3 24.5 mm to (27.9, 36.8)
- moved JP3 14.0 mm to (74.9, 15.2)
- moved JP5 12.7 mm to (30.5, 15.2)
- moved DOWN 3.81 mm to (20.3, 52.1), turned to 0 degrees
Connections:
- net N$51 renamed BUZZERPIN
- removed net N$1: LEFT.3, LEFT.4
- removed net N$10: IC1.10, JP10.10, JP3.10
- removed net N$11: IC1.11, JP6.10, JP7.10
- removed net N$12: IC1.12, JP6.9, JP7.9
- removed net N$13: IC1.13, JP6.8, JP7.8
- removed net N$14: IC1.14, JP6.7, JP7.7
- removed net N$15: IC1.15, JP6.6, JP7.6
- removed net N$16: IC1.16, JP6.5, JP7.5
- removed net N$2: LEFT.1, LEFT.2, R1.1
- removed net N$20: RIGHT.3, RIGHT.4
- removed net N$22: R2.1, RIGHT.1, RIGHT.2
- removed net N$28: IC1.31, JP5.10, JP8.10
- removed net N$29: IC1.32, JP5.9, JP8.9
- removed net N$30: IC1.33, JP5.8, JP8.8
- removed net N$35: IC1.38, JP5.3, JP8.3
- removed net N$4: IC1.2, JP10.2, JP3.2
- removed net N$43: DOWN.3, DOWN.4
- removed net N$44: DOWN.1, DOWN.2, R3.1
- removed net N$45: UP.3, UP.4
- removed net N$46: R4.1, UP.1, UP.2
- removed net N$47: SELECT.3, SELECT.4
- removed net N$48: R5.1, SELECT.1, SELECT.2
- removed net N$49: BACK.3, BACK.4
- removed net N$5: IC1.3, JP10.3, JP3.3
- removed net N$50: BACK.1, BACK.2, R6.1
- removed net N$6: IC1.4, JP10.4, JP3.4
- removed net N$7: IC1.5, JP10.5, JP3.5
- removed net N$8: IC1.8, JP10.8, JP3.8
- removed net N$9: IC1.9, JP10.9, JP3.9
- new net BACKSIG: BACK.1, BACK.2, IC1.4, JP14.7, JP14.8, R6.1
- new net BUZZER: IC1.13, JP5.15, JP5.16
- new net DOWNSIG: DOWN.1, DOWN.2, IC1.14, JP5.13, JP5.14, R3.1
- new net LEFTSIG: IC1.2, JP14.3, JP14.4, LEFT.1, LEFT.2, R1.1
- new net N$56: IC1.33, JP4.15, JP4.16
- new net N$57: IC1.34, JP4.13, JP4.14
- new net N$59: IC1.35, JP4.11, JP4.12
- new net N$63: IC1.36, JP4.10, JP4.9
- new net N$64: IC1.37, JP4.7, JP4.8
- new net N$65: IC1.38, JP4.5, JP4.6
- new net N$66: IC1.39, JP4.3, JP4.4
- new net N$67: IC1.40, JP4.1, JP4.2
- new net N$68: IC1.6, JP14.11, JP14.12
- new net N$69: IC1.27, JP3.13, JP3.14
- new net RIGHTSIG: IC1.15, JP5.11, JP5.12, R2.1, RIGHT.1, RIGHT.2
- new net SELECTSIG: IC1.3, JP14.5, JP14.6, R5.1, SELECT.1, SELECT.2
- new net UPSIG: IC1.7, JP14.13, JP14.14, R4.1, UP.1, UP.2
- net 3.3V: now also BACK.3, BACK.4, DOWN.3, DOWN.4, JP14.1, JP14.2, LEFT.3, LEFT.4, RIGHT.3, RIGHT.4, SELECT.3, SELECT.4, UP.3, UP.4; no longer JP10.1, JP3.1
- net GND: now also JP3.3, JP3.4, JP5.1, JP5.2; no longer JP4.2, JP6.1, JP7.1, JP9.2
- net N$17: now also IC1.5, JP14.10, JP14.9; no longer IC1.17, JP6.4, JP7.4
- net N$18: now also IC1.8, JP14.15, JP14.16; no longer IC1.18, JP6.3, JP7.3
- net N$19: now also IC1.9, JP14.17, JP14.18; no longer IC1.19, JP6.2, JP7.2
- net N$21: now also JP3.1, JP3.2; no longer JP4.1, JP9.1
- net N$23: now also JP3.5, JP3.6; no longer JP4.3, JP9.3
- net N$24: now also JP3.7, JP3.8; no longer JP4.4, JP9.4
- net N$25: now also IC1.10, JP14.19, JP14.20; no longer IC1.28, JP4.8, JP9.8
- net N$26: now also IC1.11, JP5.19, JP5.20; no longer IC1.29, JP4.9, JP9.9
- net N$27: now also IC1.12, JP5.17, JP5.18; no longer IC1.30, JP4.10, JP9.10
- net N$31: now also IC1.16, JP5.10, JP5.9; no longer IC1.34, JP5.7, JP8.7
- net N$32: now also IC1.17, JP5.7, JP5.8; no longer IC1.35, JP5.6, JP8.6
- net N$33: now also IC1.18, JP5.6; no longer IC1.36, JP8.5
- net N$34: now also IC1.19, JP5.3; no longer IC1.37, JP8.4
- net N$36: now also IC1.28, JP3.15, JP3.16; no longer IC1.39, JP5.2, JP8.2
- net N$37: now also IC1.29, JP3.17, JP3.18; no longer IC1.40, JP5.1, JP8.1
- net N$38: now also IC1.30, JP3.19, JP3.20; no longer IC1.6, JP10.6, JP3.6
- net N$39: now also IC1.31, JP4.19, JP4.20; no longer IC1.27, JP4.7, JP9.7
- net N$40: now also IC1.32, JP4.17, JP4.18; no longer IC1.7, JP10.7, JP3.7
- net N$41: now also JP3.11, JP3.12; no longer JP4.6, JP9.6
- net N$42: now also JP3.10, JP3.9; no longer JP4.5, JP9.5

Commit message: finished board
Parts:
- added R7: 330, rcl:0207/10
- added SJ1, SJ2: (no value), jumper:SJ
- JP1, JP2: value (none) -> Display
- moved R1 74.0 mm to (3.81, 78.7), turned to 90 degrees
- moved LS1 54.3 mm to (17.8, 82.5), turned to 270 degrees
- moved R2 41.1 mm to (25.4, 50.8), turned to 270 degrees
- moved R3 15.3 mm to (21.6, 50.8), turned to 270 degrees
- moved R4 11.5 mm to (7.62, 78.7), turned to 90 degrees
- moved RIGHT 7.73 mm to (21.6, 62.2), turned to 180 degrees
- moved R6 6.84 mm to (102.9, 72.4), turned to 90 degrees
- moved DOWN 6.84 mm to (14.0, 54.6)
- moved UP 5.24 mm to (14.0, 69.8)
- moved R5 4.58 mm to (106.7, 72.4), turned to 90 degrees
- moved LEFT 4.02 mm to (6.35, 62.2)
- moved X1 2.05 mm to (102.2, 84.6), turned to 0 degrees
- moved SELECT 1.80 mm to (109.2, 62.2), turned to 0 degrees
- moved BACK 1.27 mm to (99.1, 62.2), turned to 0 degrees
Connections:
- removed net BUZZER: IC1.13, JP5.15, JP5.16
- removed net N$18: IC1.8, JP14.15, JP14.16
- removed net N$19: IC1.9, JP14.17, JP14.18
- removed net N$25: IC1.10, JP14.19, JP14.20
- removed net N$26: IC1.11, JP5.19, JP5.20
- removed net N$27: IC1.12, JP5.17, JP5.18
- removed net N$53: X1.2
- removed net N$54: X1.3
- removed net N$63: IC1.36, JP4.10, JP4.9
- removed net N$64: IC1.37, JP4.7, JP4.8
- new net BL: JP1.7, JP2.7, R7.2
- new net RX: IC1.37, JP4.7, JP4.8, X1.2
- new net TX: IC1.36, JP4.10, JP4.9, X1.3
- net BUZZERPIN: now also IC1.13, JP5.15, JP5.16
- net CE: now also IC1.12, JP5.17, JP5.18
- net CLK: now also IC1.11, JP5.19, JP5.20
- net DC: now also IC1.9, JP14.17, JP14.18
- net DIN: now also IC1.8, JP14.15, JP14.16
- net GND: now also SJ1.1
- net LIGHT: now also R7.1, SJ1.2, SJ2.2; no longer JP1.7, JP2.7
- net N$34: now also SJ2.1
- net RESET: now also IC1.10, JP14.19, JP14.20
Routing:
- net 3.3V: track 0.00 -> 455.9 mm, vias 0 -> 1
- net LEFTSIG: track 0.00 -> 167.1 mm
- net UPSIG: track 0.00 -> 107.9 mm, vias 0 -> 2
- net BL: track 0.00 -> 106.0 mm, vias 0 -> 1
- net RESET: track 0.00 -> 104.4 mm
- net RX: track 0.00 -> 101.3 mm, vias 0 -> 1
- net TX: track 0.00 -> 100.6 mm
- net DIN: track 0.00 -> 98.8 mm
- net CLK: track 0.00 -> 86.6 mm, vias 0 -> 1
- net DC: track 0.00 -> 85.8 mm, vias 0 -> 1
- net SELECTSIG: track 0.00 -> 83.0 mm
- net CE: track 0.00 -> 75.6 mm
- net BUZZERPIN: track 0.00 -> 75.6 mm
- net BACKSIG: track 0.00 -> 73.4 mm
- net RIGHTSIG: track 0.00 -> 61.9 mm
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Other:
- outline, holes or cut-outs redrawn
